File: PicoTorch.kicad_pcb (KiCad board)
At the start: 2 copper layers, 78.7 x 62.2 mm, 44 parts, among them J1 Screw_Terminal_01x02, M1 Fan, M2 Fan, M3 Fan, M4 Fan, Q1 IRLB8721, Q2 IRLB8721, Q3 IRLB8721, Q4 IRLB8721, T1R1 4.7k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

Commit message: changes
Parts:
- added G***: LOGO, LOGO, F.Cu at (73.9, 73.6)
- added G***: LOGO, LOGO, B.Cu at (44.7, 46.1)
- D1, D3, D5, D7: footprint LED_THT:LED_D5.0mm_IRGrey -> LED_THT:LED_D1.8mm_W3.3mm_H2.4mm
- J1, M4: footprint TerminalBlock_Philmore:TerminalBlock_Philmore_TB132_1x02_P5.00mm_Horizontal -> TerminalBlock_Phoenix:TerminalBlock_Phoenix_MKDS-1,5-2_1x02_P5.00mm_Horizontal
- R1, R10, R11, R12, R2, R3, R4, R5, R6, R7, R8, R9, T1R1, T1R2, T1R3, T1R4: footprint Resistor_THT:R_Axial_DIN0204_L3.6mm_D1.6mm_P5.08mm_Horizontal -> Resistor_THT:R_Axial_DIN0207_L6.3mm_D2.5mm_P2.54mm_Vertical
- moved R7 4.47 mm to (103.0, 43.8), turned to 0 degrees
- moved R4 4.04 mm to (78.7, 43.8), turned to 0 degrees
- moved R1 3.86 mm to (54.5, 43.7), turned to 0 degrees
- moved T1R1 2.78 mm to (43.5, 83.2), turned to -90 degrees
- moved T1R2 2.78 mm to (52.6, 83.2), turned to -90 degrees
- moved T1R3 2.78 mm to (61.4, 83.2), turned to -90 degrees
- moved T1R4 2.78 mm to (70.5, 83.2), turned to -90 degrees
- moved R10 1.98 mm to (101.7, 65.0)
- moved R8 1.71 mm to (103.3, 56.9)
- moved R2 1.64 mm to (54.5, 56.8)
- moved R5 1.50 mm to (78.7, 56.8)
- moved R9 1.42 mm to (103.3, 53.8)
- moved R3 1.38 mm to (54.5, 53.7)
- moved R11 1.26 mm to (88.0, 62.3)
- moved R6 1.19 mm to (78.7, 53.7)
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Routing:
- net /Vin: track 145.3 -> 43.0 mm
- net /Thermistor3: track 27.4 -> 32.5 mm
- net /Thermistor1: track 16.6 -> 20.5 mm
- net /Thermistor2: track 20.8 -> 24.8 mm
- net +3.3V: track 38.7 -> 35.0 mm, vias 6 -> 0
- net /Mosfet3: track 44.9 -> 47.3 mm
- net /M0: track 20.5 -> 22.5 mm
- net Net-(Q2-G): track 15.3 -> 13.7 mm
- net Net-(Q1-G): track 15.3 -> 13.9 mm
- net /M2: track 61.7 -> 63.2 mm
- net Net-(Q3-G): track 15.3 -> 13.9 mm
- net Net-(D3-A): track 5.98 -> 5.07 mm
- net Net-(D7-A): track 6.02 -> 6.89 mm
- net Net-(D5-A): track 5.84 -> 5.07 mm
- net Net-(D1-A): track 5.98 -> 5.25 mm
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- added copper zone on B.Cu, net /Vin
- added copper zone on F.Cu, net /Vin
Other:
- board text added: "+"
- board text added: "+24v"
- board text added: "-"
- board text added: "GND"

Commit message: feat: First untested release
This has not been tested. It passes ERC and DRC, but zero actual
physical testing of this board has been done. It needs to be ordered
and tested to completion, as well as documenting amp limits of the
board. Please reach out if you have done any testing.
Parts:
- added SW1: SW_Push_Dual_x2, Connector_JST:JST_XH_B2B-XH-A_1x02_P2.50mm_Vertical, F.Cu at (88.7, 78.5)
- added SW2: SW_Push_Dual_x2, Connector_JST:JST_XH_B2B-XH-A_1x02_P2.50mm_Vertical, F.Cu at (95.7, 78.5)
- added SW3: SW_Push_Dual_x2, Connector_JST:JST_XH_B2B-XH-A_1x02_P2.50mm_Vertical, F.Cu at (102.6, 78.5)
- D2, D4, D6, D8: footprint Diode_THT:D_DO-201AD_P12.70mm_Horizontal -> Diode_THT:D_DO-34_SOD68_P7.62mm_Horizontal
- moved D8 6.28 mm to (96.3, 68.7)
- moved D2 2.40 mm to (60.5, 43.7)
- moved D4 2.00 mm to (85.3, 43.6)
- moved D6 1.90 mm to (109.8, 43.8)
- moved G*** 1.88 mm to (46.1, 47.4)
- moved H2 0.32 mm to (111.0, 63.2)
- moved H1 0.22 mm to (83.8, 90.5)
Connections:
- ZERO1 pad 12: unconnected-(ZERO1-11-Pad12) -> /GP11
- ZERO1 pad 13: unconnected-(ZERO1-12-Pad13) -> /GP12
- ZERO1 pad 14: unconnected-(ZERO1-13-Pad14) -> /GP13
Routing:
- net /GP11: track 0.00 -> 43.8 mm
- net /Mosfet3: track 47.3 -> 85.0 mm
- net /GP12: track 0.00 -> 35.9 mm
- net /GP13: track 0.00 -> 27.9 mm
- net /Mosfet1: track 31.6 -> 29.1 mm
- net /Vin: track 43.0 -> 45.2 mm
- net +3.3V: track 35.0 -> 37.2 mm
- net /Mosfet0: track 31.2 -> 30.6 mm
Other:
- board text added: "GP0"
- board text added: "GP1"
- board text added: "GP11"
- board text added: "GP12"
- board text added: "GP13"
- board text added: "GP2"
- board text added: "GP26"
- board text added: "GP27"
- board text added: "GP28"
- board text added: "GP29"
- board text added: "GP3"
- board text added: "UntestedAlpha1"
